File: src/kicad-250K-G-v2/kicad-250K-G-v2.sch (KiCad schematic (older format))
At the start: 28 parts, among them P1 In, P2 Out, P3 Power, U1 TL072

Commit message: final 2014-07-01
Parts:
- added C10: 100p, Custom:C2-LARGE_PADS, symbol C
Connections:
- net at C5.2, C6.2, R6.2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: now also C10.1
- net at R10.2, R7.1, R8.1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: now also C10.2
Other:
- moved on the sheet: C1, C2, C3, C4, C5, C6, C8, C9, P1, P3, R1, R11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
