File: src/kicad-100K-G-v2/_autosave-kicad-100K-G-v2.kicad_pcb (KiCad board)
At the start: 2 copper layers, 35.6 x 48.3 mm, 29 parts, among them P1 In, P2 Out, P3 Power, U1 TL072

Commit message: 28/09/2014 minor changes
Parts:
- C3: value 22n -> 10n
- C4: value 3.3n -> 1.5n
- C5: value 10n -> 6.8n
- C6: value 2.2n -> 1.5n
- R6: value 10K -> 22K
- moved R1 0.64 mm to (116.8, 116.2)
Routing:
- net Net-(P1-Pad2): track 8.67 -> 9.31 mm
- added copper zone on B.Cu, net GND
Other:
- board size 35.6 x 48.3 mm -> 35.6 x 47.6 mm
- board text added: "3eq-100k-g-v2"
- board text removed: "3eq-100k-b-v2"
