File: src/kicad-100K-B-v2/kicad-100K-B-v2.sch (KiCad schematic (older format))
At the start: 29 parts, among them P1 In, P2 Out, P3 Power, U1 TL072

Commit message: 28/09/2014 minor changes
Parts:
- R10: value 500 -> 470
- R2: value 5Meg -> 4.7 Meg
Changed lines of the file:
@@
 Sheet 1 1
 Title "Preamp 3EQ \"Lutherie Amateur\""
-Date "27 August 2014"
+Date "27 Sept 2014"
 Rev "V2"
 Comp ""
@@
 P 2450 4000
 F 0 "R2" V 2530 4000 40  0000 C CNN
-F 1 "5Meg" V 2457 4001 40  0000 C CNN
+F 1 "4.7 Meg" V 2457 4001 40  0000 C CNN
 F 2 "Custom:R3-LARGE_PADS" V 2380 4000 30  0001 C CNN
 F 3 "" H 2450 4000 30  0000 C CNN
@@
 P 7450 5850
 F 0 "R10" V 7530 5850 40  0000 C CNN
-F 1 "500" V 7457 5851 40  0000 C CNN
+F 1 "470" V 7457 5851 40  0000 C CNN
 F 2 "Custom:R3-LARGE_PADS" V 7380 5850 30  0001 C CNN
 F 3 "" H 7450 5850 30  0000 C CNN

Commit message: changes in bass version
Parts:
- C1: Ref_Mouser (none) -> 505-MKS2.1/100/10
- C10: Ref_Mouser (none) -> 505-FKP247/1000/10
- C2: Ref_Mouser (none) -> 647-UVZ1H2R2MDD
- C3: Ref_Mouser (none) -> 80-R82EC2220DQ50J
- C4: Ref_Mouser (none) -> 505-FKS23300/100/5
- C5: Ref_Mouser (none) -> 80-R82EC2100DQ50K
- C6: Ref_Mouser (none) -> 80-R82EC1220DQ50J
- C7, C9: Ref_Mouser (none) -> 667-EEU-FC1H100L
- C8: Ref_Mouser (none) -> 667-ECE-A1HKA010
- R1: Ref_Mouser (none) -> 71-CCF071K00GKE36
- R10: Ref_Mouser (none) -> 71-CCF07470RGKE36
- R11, R12: Ref_Mouser (none) -> 71-CCF07100KGKE36
- R2: Ref_Mouser (none) -> 603-MFR-25FRF52-4M7
- R3, R7: Ref_Mouser (none) -> 71-CCF0722K0GKE36
- R4, R6, R8: Ref_Mouser (none) -> 603-MFR-25FRF5210K
- R5, R9: Ref_Mouser (none) -> 71-CCF074K70GKE36
- RV1, RV2, RV3: Ref_Mouser (none) -> 652-PDB181-E420K104B
- U1: Ref_Mouser (none) -> 595-OPA2277PA
Changed lines of the file:
@@
 F 2 "Custom:DIP-8_LARGE_PADS" H 3200 3550 60  0001 C CNN
 F 3 "" H 3200 3550 60  0000 C CNN
+F 4 "595-OPA2277PA" H 3200 3550 60  0001 C CNN "Ref_Mouser"
 	1    3200 3550
 	1    0    0    -1
@@
 F 2 "Custom:R3-LARGE_PADS" V 1630 3450 30  0001 C CNN
 F 3 "" H 1700 3450 30  0000 C CNN
+F 4 "71-CCF071K00GKE36" V 1700 3450 60  0001 C CNN "Ref_Mouser"
 	1    1700 3450
 	0    1    1    0
@@
 F 2 "Custom:C2-LARGE_PADS" H 2238 3300 30  0001 C CNN
 F 3 "" H 2200 3450 60  0000 C CNN
+F 4 "505-MKS2.1/100/10" V 2200 3450 60  0001 C CNN "Ref_Mouser"
 	1    2200 3450
 	0    -1   -1   0
@@
 F 2 "Custom:R3-LARGE_PADS" V 2380 4000 30  0001 C CNN
 F 3 "" H 2450 4000 30  0000 C CNN
+F 4 "603-MFR-25FRF52-4M7" V 2450 4000 60  0001 C CNN "Ref_Mouser"
 	1    2450 4000
 	1    0    0    1
@@
 F 2 "Custom:R3-LARGE_PADS" V 4480 3550 30  0001 C CNN
 F 3 "" H 4550 3550 30  0000 C CNN
+F 4 "71-CCF0722K0GKE36" V 4550 3550 60  0001 C CNN "Ref_Mouser"
 	1    4550 3550
 	0    1    1    0
@@
 F 2 "Custom:R3-LARGE_PADS" V 4480 4300 30  0001 C CNN
 F 3 "" H 4550 4300 30  0000 C CNN
+F 4 "603-MFR-25FRF5210K" V 4550 4300 60  0001 C CNN "Ref_Mouser"
 	1    4550 4300
 	0    1    1    0
@@
 F 2 "Custom:R3-LARGE_PADS" V 6030 4900 30  0001 C CNN
 F 3 "" H 6100 4900 30  0000 C CNN
+F 4 "71-CCF074K70GKE36" V 6100 4900 60  0001 C CNN "Ref_Mouser"
 	1    6100 4900
 	0    1    1    0
@@
 F 3 "" H 5200 3550 60  0000 C CNN
 F 4 "Low" H 5000 3400 60  0000 C CNN "Field4"
+F 5 "652-PDB181-E420K104B" H 5200 3550 60  0001 C CNN "Ref_Mouser"
 	1    5200 3550
 	-1   0    0    1
@@
 F 2 "Custom:C2-LARGE_PADS" H 5238 3100 30  0001 C CNN
 F 3 "" H 5200 3250 60  0000 C CNN
+F 4 "80-R82EC2220DQ50J" V 5200 3250 60  0001 C CNN "Ref_Mouser"
 	1    5200 3250
 	0    -1   -1   0
@@
 F 2 "Custom:R3-LARGE_PADS" V 6030 3550 30  0001 C CNN
 F 3 "" H 6100 3550 30  0000 C CNN
+F 4 "71-CCF0722K0GKE36" V 6100 3550 60  0001 C CNN "Ref_Mouser"
 	1    6100 3550
 	0    1    1    0
@@
 F 2 "Custom:C2-LARGE_PADS" H 5238 3850 30  0001 C CNN
 F 3 "" H 5200 4000 60  0000 C CNN
+F 4 "505-FKS23300/100/5 " V 5200 4000 60  0001 C CNN "Ref_Mouser"
 	1    5200 4000
 	0    -1   -1   0
@@
 F 3 "" H 5200 4300 60  0000 C CNN
 F 4 "Mid" H 5000 4150 60  0000 C CNN "Field4"
+F 5 "652-PDB181-E420K104B" H 5200 4300 60  0001 C CNN "Ref_Mouser"
 	1    5200 4300
 	-1   0    0    1
@@
 F 2 "Custom:R3-LARGE_PADS" V 6030 4300 30  0001 C CNN
 F 3 "" H 6100 4300 30  0000 C CNN
+F 4 "603-MFR-25FRF5210K" V 6100 4300 60  0001 C CNN "Ref_Mouser"
 	1    6100 4300
 	0    1    1    0
@@
 F 2 "Custom:R3-LARGE_PADS" V 5430 3750 30  0001 C CNN
 F 3 "" H 5500 3750 30  0000 C CNN
+F 4 "603-MFR-25FRF5210K" V 5500 3750 60  0001 C CNN "Ref_Mouser"
 	1    5500 3750
 	0    -1   -1   0
@@
 F 3 "" H 5200 4900 60  0000 C CNN
 F 4 "High" H 4950 4750 60  0000 C CNN "Field4"
+F 5 "652-PDB181-E420K104B" H 5200 4900 60  0001 C CNN "Ref_Mouser"
 	1    5200 4900
 	-1   0    0    1
@@
 F 2 "Custom:C2-LARGE_PADS" H 5588 4400 30  0001 C CNN
 F 3 "" H 5550 4550 60  0000 C CNN
+F 4 "80-R82EC2100DQ50K" V 5550 4550 60  0001 C CNN "Ref_Mouser"
 	1    5550 4550
 	0    -1   -1   0
@@
 F 2 "Custom:R3-LARGE_PADS" V 4480 4900 30  0001 C CNN
 F 3 "" H 4550 4900 30  0000 C CNN
+F 4 "71-CCF074K70GKE36" V 4550 4900 60  0001 C CNN "Ref_Mouser"
 	1    4550 4900
 	0    1    1    0
@@
 F 2 "Custom:C2-LARGE_PADS" H 5588 5000 30  0001 C CNN
 F 3 "" H 5550 5150 60  0000 C CNN
+F 4 "80-R82EC1220DQ50J " V 5550 5150 60  0001 C CNN "Ref_Mouser"
 	1    5550 5150
 	0    -1   -1   0
@@
 F 2 "Custom:R3-LARGE_PADS" V 7380 5850 30  0001 C CNN
 F 3 "" H 7450 5850 30  0000 C CNN
+F 4 "71-CCF07470RGKE36" V 7450 5850 60  0001 C CNN "Ref_Mouser"
 	1    7450 5850
 	0    1    1    0
@@
 F 2 "Custom:C1.5V7-LARGE_PADS" H 7950 5850 60  0001 C CNN
 F 3 "" H 7950 5850 60  0000 C CNN
+F 4 "667-EEU-FC1H100L" H 7950 5850 60  0001 C CNN "Ref_Mouser"
 	1    7950 5850
 	0    -1   -1   0
@@
 F 2 "Custom:R3-LARGE_PADS" V 9080 4200 30  0001 C CNN
 F 3 "" H 9150 4200 30  0000 C CNN
+F 4 "71-CCF07100KGKE36" V 9150 4200 60  0001 C CNN "Ref_Mouser"
 	1    9150 4200
 	1    0    0    1
@@
 F 2 "Custom:R3-LARGE_PADS" V 9080 4900 30  0001 C CNN
 F 3 "" H 9150 4900 30  0000 C CNN
+F 4 "71-CCF07100KGKE36" V 9150 4900 60  0001 C CNN "Ref_Mouser"
 	1    9150 4900
 	1    0    0    1
@@
 F 2 "Custom:C1.5V7-LARGE_PADS" H 9450 4900 60  0001 C CNN
 F 3 "" H 9450 4900 60  0000 C CNN
+F 4 "667-ECE-A1HKA010" H 9450 4900 60  0001 C CNN "Ref_Mouser"
 	1    9450 4900
 	1    0    0    -1
@@
 F 2 "Custom:C1.5V7-LARGE_PADS" H 9750 4550 60  0001 C CNN
 F 3 "" H 9750 4550 60  0000 C CNN
+F 4 "667-EEU-FC1H100L" H 9750 4550 60  0001 C CNN "Ref_Mouser"
 	1    9750 4550
 	1    0    0    -1
@@
 F 2 "Custom:C1.5V7-LARGE_PADS" H 4000 3550 60  0001 C CNN
 F 3 "" H 4000 3550 60  0000 C CNN
+F 4 "647-UVZ1H2R2MDD" H 4000 3550 60  0001 C CNN "Ref_Mouser"
 	1    4000 3550
 	0    -1   -1   0
@@
 F 2 "Custom:C2-LARGE_PADS" H 6288 5000 30  0001 C CNN
 F 3 "" H 6250 5150 60  0000 C CNN
+F 4 "505-FKP247/1000/10" V 6250 5150 60  0001 C CNN "Ref_Mouser"
 	1    6250 5150
 	0    -1   -1   0
